File: KiCad/filter3.kicad_sch (KiCad schematic)
At the start: 14 parts, among them J1 Screw_Terminal_01x02, J2 Screw_Terminal_01x02, J5 Screw_Terminal_01x02, J6 Screw_Terminal_01x02, U1 NE5532

Commit message: nya filtret
Parts:
- removed J1: Screw_Terminal_01x02, TerminalBlock:TerminalBlock_MaiXu_MX126-5.0-02P_1x02_P5.00mm, symbol Connector:Screw_Terminal_01x02
- R1: value 18k -> 12k
- R2: value 18k -> 3.9k
- R3, R7: value 1.3k -> 3.3k
Connections:
- net 4.5V is gone; now on net GND: C3.2
- net GND: now also R2.1
- no-connect marks 1 -> 0
Changed lines of the file:
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@@
+	)
+	(junction
+		(at 137.16 83.82)
+		(diameter 0)
+		(color 0 0 0 0)
+	)
+	(junction
+		(at 85.09 109.22)
+		(diameter 0)
+		(color 0 0 0 0)
+	)
+	(junction
+		(at 110.49 81.28)
+		(diameter 0)
+		(color 0 0 0 0)
+	)
+	(junction
+		(at 81.28 143.51)
+		(diameter 0)
+		(color 0 0 0 0)
+	)
+	(junction
+		(at 208.28 83.82)
+		(diameter 0)
+		(color 0 0 0 0)
+	)
+	(junction
+		(at 85.09 111.76)
+		(diameter 0)
+		(color 0 0 0 0)
 	)
 	(junction
@@
 		(color 0 0 0 0)
 	)
-	(junction
-		(at 137.16 83.82)
-		(diameter 0)
-		(color 0 0 0 0)
-	)
-	(junction
-		(at 85.09 109.22)
-		(diameter 0)
-		(color 0 0 0 0)
-	)
-	(junction
-		(at 110.49 81.28)
-		(diameter 0)
-		(color 0 0 0 0)
-	)
-	(junction
-		(at 81.28 143.51)
-		(diameter 0)
-		(color 0 0 0 0)
-	)
-	(junction
-		(at 208.28 83.82)
-		(diameter 0)
-		(color 0 0 0 0)
-	)
-	(junction
-		(at 85.09 111.76)
-		(diameter 0)
-		(color 0 0 0 0)
-	)
-	(no_connect
-		(at 237.49 86.36)
-	)
 	(wire
 		(pts
@@
 	(wire
 		(pts
+			(xy 232.41 86.36) (xy 241.3 86.36)
+		)
+		(stroke
+			(width 0)
+			(type default)
+		)
+	)
+	(wire
+		(pts
 			(xy 149.86 83.82) (xy 168.91 83.82)
 		)
@@
 	(wire
 		(pts
+			(xy 100.33 66.04) (xy 110.49 66.04)
+		)
+		(stroke
+			(width 0)
+			(type default)
+		)
+	)
+	(wire
+		(pts
 			(xy 137.16 111.76) (xy 116.84 111.76)
 		)
@@
 	(wire
 		(pts
-			(xy 232.41 86.36) (xy 241.3 86.36)
+			(xy 203.2 64.77) (xy 208.28 64.77)
 		)
 		(stroke
@@
 	(wire
 		(pts
-			(xy 36.83 36.83) (xy 36.83 40.64)
-		)
-		(stroke
-			(width 0)
-			(type default)
-		)
-	)
-	(wire
-		(pts
 			(xy 191.77 83.82) (xy 208.28 83.82)
 		)
@@
 			(width 0)
 			(type default)
-		)
-	)
-	(global_label "4.5V"
-		(shape input)
-		(at 208.28 64.77 90)
-		(fields_autoplaced yes)
-		(effects
-			(font
-				(size 1.27 1.27)
-			)
-			(justify left)
-		)
-		(property "Intersheetrefs" "${INTERSHEET_REFS}"
-			(at 208.28 57.6724 90)
-			(effects
-				(font
-					(size 1.27 1.27)
-				)
-				(justify left)
-				(hide yes)
-			)
 		)
 	)
@@
 		)
 	)
-	(global_label "4.5V"
-		(shape input)
-		(at 36.83 34.29 180)
-		(fields_autoplaced yes)
-		(effects
-			(font
-				(size 1.27 1.27)
-			)
-			(justify right)
-		)
-		(property "Intersheetrefs" "${INTERSHEET_REFS}"
-			(at 29.7324 34.29 0)
-			(effects
-				(font
-					(size 1.27 1.27)
-				)
-				(justify right)
-				(hide yes)
-			)
-		)
-	)
 	(global_label "+9V"
 		(shape input)
@@
 				)
 				(justify right)
-				(hide yes)
-			)
-		)
-	)
-	(global_label "4.5V"
-		(shape input)
-		(at 110.49 64.77 90)
-		(fields_autoplaced yes)
-		(effects
-			(font
-				(size 1.27 1.27)
-			)
-			(justify left)
-		)
-		(property "Intersheetrefs" "${INTERSHEET_REFS}"
-			(at 110.49 57.6724 90)
-			(effects
-				(font
-					(size 1.27 1.27)
-				)
-				(justify left)
 				(hide yes)
 			)
@@
 			)
 		)
-		(property "Value" "18k"
+		(property "Value" "3.9k"
 			(at 106.172 75.184 0)
 			(effects
@@
 				(path "/915b7235-ddd1-4a9f-82e1-c7cfdeb31b6c"
 					(reference "R2")
-					(unit 1)
-				)
-			)
-		)
-	)
-	(symbol
-		(lib_id "Connector:Screw_Terminal_01x02")
-		(at 41.91 34.29 0)
-		(unit 1)
-		(exclude_from_sim no)
-		(in_bom yes)
-		(on_board yes)
-		(dnp no)
-		(fields_autoplaced yes)
-		(property "Reference" "J1"
-			(at 44.45 34.2899 0)
-			(effects
-				(font
-					(size 1.27 1.27)
-				)
-				(justify left)
-			)
-		)
-		(property "Value" "Screw_Terminal_01x02"
-			(at 44.45 36.8299 0)
-			(effects
-				(font
-					(size 1.27 1.27)
-				)
-				(justify left)
-				(hide yes)
-			)
-		)
-		(property "Footprint" "TerminalBlock:TerminalBlock_MaiXu_MX126-5.0-02P_1x02_P5.00mm"
-			(at 41.91 34.29 0)
-			(effects
-				(font
-					(size 1.27 1.27)
-				)
-				(hide yes)
-			)
-		)
-		(property "Datasheet" "~"
-			(at 41.91 34.29 0)
-			(effects
-				(font
-					(size 1.27 1.27)
-				)
-				(hide yes)
-			)
-		)
-		(property "Description" "Generic screw terminal, single row, 01x02, script generated (kicad-library-utils/schlib/autogen/connector/)"
-			(at 41.91 34.29 0)
-			(effects
-				(font
-					(size 1.27 1.27)
-				)
-				(hide yes)
-			)
-		)
-		(pin "1"
-		)
-		(pin "2"
-		)
-		(instances
-			(project ""
-				(path "/915b7235-ddd1-4a9f-82e1-c7cfdeb31b6c"
-					(reference "J1")
 					(unit 1)
 				)
@@
 	)
 	(symbol
+		(lib_id "power:GND")
+		(at 203.2 64.77 0)
+		(unit 1)
+		(exclude_from_sim no)
+		(in_bom yes)
+		(on_board yes)
+		(dnp no)
+		(fields_autoplaced yes)
+		(property "Reference" "#PWR06"
+			(at 203.2 71.12 0)
+			(effects
+				(font
+					(size 1.27 1.27)
+				)
+				(hide yes)
+			)
+		)
+		(property "Value" "GND"
+			(at 203.2 69.85 0)
+			(effects
+				(font
+					(size 1.27 1.27)
+				)
+			)
+		)
+		(property "Footprint" ""
+			(at 203.2 64.77 0)
+			(effects
+				(font
+					(size 1.27 1.27)
+				)
+				(hide yes)
+			)
+		)
+		(property "Datasheet" ""
+			(at 203.2 64.77 0)
+			(effects
+				(font
+					(size 1.27 1.27)
+				)
+				(hide yes)
+			)
+		)
+		(property "Description" "Power symbol creates a global label with name \"GND\" , ground"
+			(at 203.2 64.77 0)
+			(effects
+				(font
+					(size 1.27 1.27)
+				)
+				(hide yes)
+			)
+		)
+		(pin "1"
+		)
+		(instances
+			(project ""
+				(path "/915b7235-ddd1-4a9f-82e1-c7cfdeb31b6c"
+					(reference "#PWR06")
+					(unit 1)
+				)
+			)
+		)
+	)
+	(symbol
 		(lib_id "power:VAC")
 		(at 81.28 151.13 180)
@@
 			)
 		)
-		(property "Value" "18k"
+		(property "Value" "12k"
 			(at 112.268 115.316 90)
 			(effects
@@
 			)
 		)
-		(property "Value" "1.3k"
+		(property "Value" "3.3k"
 			(at 187.96 86.614 90)
 			(effects
@@
 			)
 		)
-		(property "Value" "1.3k"
+		(property "Value" "3.3k"
 			(at 146.05 86.614 90)
 			(effects
@@
 	(symbol
 		(lib_id "power:GND")
-		(at 36.83 40.64 0)
+		(at 100.33 66.04 0)
 		(unit 1)
 		(exclude_from_sim no)
@@
 		(dnp no)
 		(fields_autoplaced yes)
-		(property "Reference" "#PWR01"
-			(at 36.83 46.99 0)
+		(property "Reference" "#PWR07"
+			(at 100.33 72.39 0)
 			(effects
 				(font
@@
 		)
 		(property "Value" "GND"
-			(at 36.83 45.72 0)
+			(at 100.33 71.12 0)
 			(effects
 				(font
@@
 		)
 		(property "Footprint" ""
-			(at 36.83 40.64 0)
+			(at 100.33 66.04 0)
 			(effects
 				(font
@@
 		)
 		(property "Datasheet" ""
-			(at 36.83 40.64 0)
+			(at 100.33 66.04 0)
 			(effects
 				(font
@@
 		)
 		(property "Description" "Power symbol creates a global label with name \"GND\" , ground"
-			(at 36.83 40.64 0)
+			(at 100.33 66.04 0)
 			(effects
 				(font
@@
 			(project ""
 				(path "/915b7235-ddd1-4a9f-82e1-c7cfdeb31b6c"
-					(reference "#PWR01")
+					(reference "#PWR07")
 					(unit 1)
 				)
