File: KiCad/filter3.kicad_pcb (KiCad board)
At the start: 2 copper layers, 14 parts, among them U1 NE5532

Commit message: nya filtret
Parts:
- removed 4.5V: Screw_Terminal_01x02, TerminalBlock:TerminalBlock_MaiXu_MX126-5.0-02P_1x02_P5.00mm
- J2: renamed from Output; value output -> Screw_Terminal_01x02
- J5: renamed from +9v; value +9v -> Screw_Terminal_01x02
- Je1: renamed from -9v; value -9v -> Screw_Terminal_01x02
- R1: value 18k -> 12k
- R2: value 18k -> 3.9k
- R3, R7: value 1.3k -> 3.3k
- renumbered input to J6
Connections:
- C3 pad 2: 4.5V -> GND
- R2 pad 1: unconnected-(R2-Pad1) -> GND
Routing:
- net GND: track 121.5 -> 136.9 mm
- net 4.5V: track 12.3 -> 0.00 mm
- net (no net): track 3.08 -> 0.00 mm
- net Net-(U1B--): track 26.1 -> 28.9 mm
Other:
- board outline added: 83.2 x 53.7 mm

Commit message: filter3
Parts:
- removed J2, J5, J6, Je1: Screw_Terminal_01x02, TerminalBlock:TerminalBlock_MaiXu_MX126-5.0-02P_1x02_P5.00mm
- added +9V: Screw_Terminal_01x02, TerminalBlock:TerminalBlock_MaiXu_MX126-5.0-02P_1x02_P5.00mm, F.Cu at (116.8, 105.5)
- added -9V: -9V, TerminalBlock:TerminalBlock_MaiXu_MX126-5.0-02P_1x02_P5.00mm, F.Cu at (136.8, 68.5)
- added Input: Screw_Terminal_01x02, TerminalBlock:TerminalBlock_MaiXu_MX126-5.0-02P_1x02_P5.00mm, F.Cu at (105.5, 105.0)
- added Output: Output, TerminalBlock:TerminalBlock_MaiXu_MX126-5.0-02P_1x02_P5.00mm, F.Cu at (159.0, 75.8)
- moved R2 45.5 mm to (110.5, 67.0), turned to 0 degrees
- moved C2 40.3 mm to (97.7, 73.7)
- moved C1 28.6 mm to (105.2, 95.0), turned to 90 degrees
- moved R1 27.8 mm to (110.5, 80.0)
- moved U1 17.7 mm to (124.2, 81.5), turned to 180 degrees
- moved C4 16.9 mm to (133.8, 82.0), turned to -90 degrees
- moved C3 13.5 mm to (143.8, 90.2), turned to 0 degrees
- moved R3 12.0 mm to (138.0, 90.2)
- moved R7 3.71 mm to (140.5, 97.0), turned to 180 degrees
Routing:
- net GND: track 136.9 -> 266.1 mm
- net -9V: track 56.5 -> 16.6 mm
- net Net-(U1B--): track 28.9 -> 55.4 mm
- net +9V: track 40.1 -> 24.0 mm
- net Signal: track 33.0 -> 48.4 mm
- net Net-(U1A-+): track 17.3 -> 30.3 mm
- net Net-(C1-Pad2): track 9.07 -> 18.5 mm
- net VAC: track 18.0 -> 10.1 mm
- net Net-(U1B-+): track 13.5 -> 10.8 mm
- net Net-(C4-Pad2): track 8.49 -> 11.0 mm
Other:
- board text removed: "Input"
